File: sf.sch (KiCad schematic (older format))
At the start: 55 parts, among them J1 DRIVE, J2 PDI, J3 AUDIO, J4 PROBE, J5 UART, Q1 IRLML6402, Q2 FDV301N, Q3 IRLML6402, SW1 OFF, SW2 ON/RANGE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

Commit message: Add notes for rev B
- Quieter inductor
- ADC reference is VCC/1.6, account for that in volpot
- Volume pot sucks
Other:
- note added: "CHANGE FOR REV B:\n\n- Quieter inductor\n- ADC reference is VCC/1.6, account for that in volpot\n- Volume pot sucks"
Changed lines of the file:
@@
 	6200 1400 6300 1400
 Connection ~ 6300 1400
+Text Notes 6600 6900 0    60   ~ 0
+CHANGE FOR REV B:\n\n- Quieter inductor\n- ADC reference is VCC/1.6, account for that in volpot\n- Volume pot sucks
 $EndSCHEMATC

Commit message: Update assembly instructions and schematic notes
Other:
- note added: "CHANGE FOR REV B:\n\n- Quieter inductor\n- C0G 1.5nF capacitors\n- ADC reference is VCC/1.6, account for that in volpot\n- Volume pot sucks\n- Fix or remove gain selection\n- Fix excess output-input coupling\n- Series resistor on UART RX"
- note removed: "CHANGE FOR REV B:\n\n- Quieter inductor\n- ADC reference is VCC/1.6, account for that in volpot\n- Volume pot sucks"
Changed lines of the file:
@@
 	6200 1400 6300 1400
 Connection ~ 6300 1400
-Text Notes 6600 6900 0    60   ~ 0
-CHANGE FOR REV B:\n\n- Quieter inductor\n- ADC reference is VCC/1.6, account for that in volpot\n- Volume pot sucks
+Text Notes 6300 7000 0    60   ~ 0
+CHANGE FOR REV B:\n\n- Quieter inductor\n- C0G 1.5nF capacitors\n- ADC reference is VCC/1.6, account for that in volpot\n- Volume pot sucks\n- Fix or remove gain selection\n- Fix excess output-input coupling\n- Series resistor on UART RX
 $EndSCHEMATC
